Commit message: simple x-orientation controller

File: description/description/urdf/model.urdf.xacro (robot description, xacro)
@@ -96,5 +96,6 @@
       <mass value="9.0877"/>
       <origin xyz="0 0 0"/>
-      <inertia ixx="0.1454" ixy="0.0" ixz="0.0" iyy="0.1366" iyz="0.0" izz="0.1594"/>
+      <!--<inertia ixx="0.1454" ixy="0.0" ixz="0.0" iyy="0.1366" iyz="0.0" izz="0.1594"/>-->
+      <inertia ixx="0.1454" ixy="0.0" ixz="0.0" iyy="1.1366" iyz="0.0" izz="1.1594"/>
     </inertial>
   </link>

Commit message: initial version of position control

File: description/description/urdf/model.urdf.xacro (robot description, xacro)
@@ -97,5 +97,5 @@
       <origin xyz="0 0 0"/>
       <!--<inertia ixx="0.1454" ixy="0.0" ixz="0.0" iyy="0.1366" iyz="0.0" izz="0.1594"/>-->
-      <inertia ixx="0.1454" ixy="0.0" ixz="0.0" iyy="1.1366" iyz="0.0" izz="1.1594"/>
+      <inertia ixx="0.1454" ixy="0.0" ixz="0.0" iyy="0.1366" iyz="0.0" izz="0.1594"/>
     </inertial>
   </link>

Commit message: first test with changing inertia

File: description/description/urdf/model.urdf.xacro (robot description, xacro)
@@ -105,4 +105,25 @@
     <child link="inertial_link" />
   </joint>
+  <link name="printed_part">
+    <self_collide>false</self_collide>
+    <visual name="printed_part_visual">
+      <origin xyz="0 0 0" rpy="0 0 0" />
+      <geometry>
+        <cylinder length="0.4" radius="0.01"/>
+      </geometry>
+    </visual>
+    <inertial>
+      <mass value="1.0"/>
+      <origin xyz="0.4 0 0"/>
+      <inertia ixx="0.01" ixy="0.0" ixz="0.0" iyy="0.01" iyz="0.0" izz="0.01"/>
+    </inertial>
+  </link>
+  <joint name="printed_joint" type="prismatic">
+    <axis xyz="0 0 1"/>
+    <origin xyz="0.8 0 0" rpy="0 1.57075 0" />
+    <parent link="body" />
+    <child link="printed_part" />
+    <limit effort="1.0" lower="-0.01" upper="0.0" velocity="0.05"/>
+  </joint>
   <gazebo>
         <plugin name="gazebo_model_plugin_mass_controller" filename="libgazebo_model_plugin_mass_controller.so">

Commit message: mid-work on visualisation

File: description/description/urdf/model.urdf.xacro (robot description, xacro)
@@ -115,5 +115,5 @@
     <inertial>
       <mass value="1.0"/>
-      <origin xyz="0.4 0 0"/>
+      <origin xyz="0.5 0 0"/>
       <inertia ixx="0.01" ixy="0.0" ixz="0.0" iyy="0.01" iyz="0.0" izz="0.01"/>
     </inertial>
@@ -121,12 +121,35 @@
   <joint name="printed_joint" type="prismatic">
     <axis xyz="0 0 1"/>
-    <origin xyz="0.8 0 0" rpy="0 1.57075 0" />
+    <origin xyz="0.2 0 0" rpy="0 1.57075 0" />
     <parent link="body" />
     <child link="printed_part" />
-    <limit effort="1.0" lower="-0.01" upper="0.0" velocity="0.05"/>
+    <limit effort="1.0" lower="-0.01" upper="0.01" velocity="0.05"/>
+  </joint>
+  <link name="print_roll">
+    <self_collide>false</self_collide>
+    <inertial>
+      <mass value="0.01"/>
+      <origin xyz="0 0 0"/>
+      <inertia ixx="0.01" ixy="0.0" ixz="0.0" iyy="0.01" iyz="0.0" izz="0.01"/>
+    </inertial>
+  </link>
+  <joint name="roll_joint" type="fixed">
+    <origin xyz="0.0 0 0" rpy="0 0 0" />
+    <parent link="body" />
+    <child link="print_roll" />
   </joint>
   <gazebo>
         <plugin name="gazebo_model_plugin_mass_controller" filename="libgazebo_model_plugin_mass_controller.so">
             <name_link_to_change_mass>body</name_link_to_change_mass>
+        </plugin>
+  </gazebo>
+  <gazebo>
+        <plugin name="gazebo_model_plugin_printing" filename="libgazebo_model_plugin_printing.so">
+            <name_link_to_print>printed_part</name_link_to_print>
+            <name_link_printing_roll>print_roll</name_link_printing_roll>
+        </plugin>
+  </gazebo>
+  <gazebo>
+        <plugin name="gazebo_visual_plugin_printing" filename="libgazebo_visual_plugin_printing.so">
         </plugin>
   </gazebo>

Commit message: visualitation update - work in progress

File: description/description/urdf/model.urdf.xacro (robot description, xacro)
@@ -110,11 +110,11 @@
       <origin xyz="0 0 0" rpy="0 0 0" />
       <geometry>
-        <cylinder length="0.4" radius="0.01"/>
+        <cylinder length="0.01" radius="0.01"/>
       </geometry>
     </visual>
     <inertial>
-      <mass value="1.0"/>
+      <mass value="0.001"/>
       <origin xyz="0.5 0 0"/>
-      <inertia ixx="0.01" ixy="0.0" ixz="0.0" iyy="0.01" iyz="0.0" izz="0.01"/>
+      <inertia ixx="0.001" ixy="0.0" ixz="0.0" iyy="0.001" iyz="0.0" izz="0.001"/>
     </inertial>
   </link>
@@ -124,5 +124,5 @@
     <parent link="body" />
     <child link="printed_part" />
-    <limit effort="1.0" lower="-0.01" upper="0.01" velocity="0.05"/>
+    <limit effort="1.0" lower="-0.01" upper="0.01" velocity="0.005"/>
   </joint>
   <link name="print_roll">
@@ -148,8 +148,4 @@
             <name_link_to_print>printed_part</name_link_to_print>
             <name_link_printing_roll>print_roll</name_link_printing_roll>
-        </plugin>
-  </gazebo>
-  <gazebo>
-        <plugin name="gazebo_visual_plugin_printing" filename="libgazebo_visual_plugin_printing.so">
         </plugin>
   </gazebo>

Commit message: working printing with visualisation

File: description/description/urdf/model.urdf.xacro (robot description, xacro)
@@ -116,13 +116,14 @@
       <mass value="0.001"/>
       <origin xyz="0.5 0 0"/>
-      <inertia ixx="0.001" ixy="0.0" ixz="0.0" iyy="0.001" iyz="0.0" izz="0.001"/>
+      <inertia ixx="0.01" ixy="0.0" ixz="0.0" iyy="0.01" iyz="0.0" izz="0.01"/>
     </inertial>
   </link>
   <joint name="printed_joint" type="prismatic">
     <axis xyz="0 0 1"/>
-    <origin xyz="0.2 0 0" rpy="0 1.57075 0" />
+    <origin xyz="0.17 0 0" rpy="0 1.57075 0" />
     <parent link="body" />
     <child link="printed_part" />
-    <limit effort="1.0" lower="-0.01" upper="0.01" velocity="0.005"/>
+    <limit effort="1.0" lower="-1.0" upper="1.0" velocity="0.001"/>
+    <dynamics friction="0.9" damping="0.9"/>
   </joint>
   <link name="print_roll">

Commit message: PID V2.0

File: description/description/urdf/model.urdf.xacro (robot description, xacro)
@@ -116,5 +116,5 @@
       <mass value="0.001"/>
       <origin xyz="0.5 0 0"/>
-      <inertia ixx="0.01" ixy="0.0" ixz="0.0" iyy="0.01" iyz="0.0" izz="0.01"/>
+      <inertia ixx="0.001" ixy="0.0" ixz="0.0" iyy="0.001" iyz="0.0" izz="0.001"/>
     </inertial>
   </link>

Commit message: 3d printing project V1.0 (#1)
* disable default ctl module and add mass modifier plugin

* add basic controller

* initial version of go and stop controller

* simple x-orientation controller

* reduce MLP workload

* further mlp workload reduction

* initial version of position control

* first test with changing inertia

* mid-work on visualisation

* visualitation update - work in progress

* working printing with visualisation

* controller testing

* test framework preparation

* mid-work - controller testing script

* controller listen to external target, ctl test module hadles communication and publish test trajectory

* full test logging

* initial version of the ctl testing framework

* improvements to testing framework

* test framework further improvements

* handling time exception

* refactor ctl scripts

* changes before PID testing

* PID V2.0

* first LQR iteration - just position control

* change orientation controller to LQR

* add test case: printing with stationary end while rotating

* Astrobee 3D printing V1.0

File: description/description/urdf/model.urdf.xacro (robot description, xacro)
@@ -96,4 +96,5 @@
       <mass value="9.0877"/>
       <origin xyz="0 0 0"/>
+      <!--<inertia ixx="0.1454" ixy="0.0" ixz="0.0" iyy="0.1366" iyz="0.0" izz="0.1594"/>-->
       <inertia ixx="0.1454" ixy="0.0" ixz="0.0" iyy="0.1366" iyz="0.0" izz="0.1594"/>
     </inertial>
@@ -104,4 +105,50 @@
     <child link="inertial_link" />
   </joint>
+  <link name="printed_part">
+    <self_collide>false</self_collide>
+    <visual name="printed_part_visual">
+      <origin xyz="0 0 0" rpy="0 0 0" />
+      <geometry>
+        <cylinder length="0.01" radius="0.01"/>
+      </geometry>
+    </visual>
+    <inertial>
+      <mass value="0.001"/>
+      <origin xyz="0.5 0 0"/>
+      <inertia ixx="0.001" ixy="0.0" ixz="0.0" iyy="0.001" iyz="0.0" izz="0.001"/>
+    </inertial>
+  </link>
+  <joint name="printed_joint" type="prismatic">
+    <axis xyz="0 0 1"/>
+    <origin xyz="0.17 0 0" rpy="0 1.57075 0" />
+    <parent link="body" />
+    <child link="printed_part" />
+    <limit effort="1.0" lower="-1.0" upper="1.0" velocity="0.001"/>
+    <dynamics friction="0.9" damping="0.9"/>
+  </joint>
+  <link name="print_roll">
+    <self_collide>false</self_collide>
+    <inertial>
+      <mass value="0.01"/>
+      <origin xyz="0 0 0"/>
+      <inertia ixx="0.01" ixy="0.0" ixz="0.0" iyy="0.01" iyz="0.0" izz="0.01"/>
+    </inertial>
+  </link>
+  <joint name="roll_joint" type="fixed">
+    <origin xyz="0.0 0 0" rpy="0 0 0" />
+    <parent link="body" />
+    <child link="print_roll" />
+  </joint>
+  <gazebo>
+        <plugin name="gazebo_model_plugin_mass_controller" filename="libgazebo_model_plugin_mass_controller.so">
+            <name_link_to_change_mass>body</name_link_to_change_mass>
+        </plugin>
+  </gazebo>
+  <gazebo>
+        <plugin name="gazebo_model_plugin_printing" filename="libgazebo_model_plugin_printing.so">
+            <name_link_to_print>printed_part</name_link_to_print>
+            <name_link_printing_roll>print_roll</name_link_printing_roll>
+        </plugin>
+  </gazebo>
   <!-- MODEL -->
   <xacro:include filename="$(find description)/urdf/model_drag.urdf.xacro" />
